File: TE0890/local_board/TE0890_etc.sch (KiCad schematic (older format))
At the start: 3 parts

Commit message: First prototype
Parts:
- added C1: 10u, Capacitor_SMD:C_0805_2012Metric_Pad1.18x1.45mm_HandSolder, symbol Device:C
- added D1, D2: LED, Capacitor_SMD:C_0805_2012Metric_Pad1.18x1.45mm_HandSolder, symbol Device:LED
- added D3: PRTR5V0U2X,215, LibraryLoader:PRTR5V0U2X, symbol LibraryLoader:PRTR5V0U2X,215
- added J10, J11, J12, J9: Conn_01x01, TestPoint:TestPoint_THTPad_D2.0mm_Drill1.0mm, symbol Connector_Generic:Conn_01x01
- added J13: 1734035-1, LibraryLoader:17340351, symbol LibraryLoader:1734035-1
- added R1, R2: 0, Resistor_SMD:R_0805_2012Metric_Pad1.20x1.40mm_HandSolder, symbol Device:R
- added R3, R4: 82, Resistor_SMD:R_0805_2012Metric_Pad1.20x1.40mm_HandSolder, symbol Device:R
- added R5, R7: 15k, Resistor_SMD:R_0805_2012Metric_Pad1.20x1.40mm_HandSolder, symbol Device:R
- added R6: 1.5k, Resistor_SMD:R_0805_2012Metric_Pad1.20x1.40mm_HandSolder, symbol Device:R
- U2, U4: renamed from U?; footprint (none) -> Connector_PinHeader_2.54mm:PinHeader_1x06_P2.54mm_Vertical
- U3: renamed from U?; footprint (none) -> TE0890:TE0790
Connections:
- net GND: now reaches U3.1 (GND)
- net GND: now also U2.2 (GND), U3.2 (GND), U3.GND, U4.1 (GND), C1.2, D1.1 (K), D2.1 (K), D3.1 (ground), J13.5, R5.2, R7.2
- net at U3.10 (TDI): now also R2.1
- net at U3.11 (Button): now also J11.1 (Pin_1)
- net at U3.12 (TMS): now also U2.6 (TMS)
- net at U3.3 (RXD): now also U4.4 (FTDI_1)
- net at U3.4 (TCK): now also U2.3 (TCK)
- net at U3.5 (3V3): now also R3.1
- net +3V3: now reaches U3.6 (VIO)
- net +3V3: now also U2.1 (3V3), R6.1
- net at U3.7 (TXD): now also U4.2 (FTDI_0)
- net at U3.8 (TDO): now also R1.1
- net at U3.9 (LED): now also J12.1 (Pin_1)
- net +5V: now reaches U4.3 (5V0)
- net +5V: now also D3.4 (supply_voltage), J13.1, R4.1
- net at U4.5 (FTDI_2): now also J9.1 (Pin_1)
- net at U4.6 (FTDI_3): now also J10.1 (Pin_1)
- net at U2.4 (TDO): now also R1.2
- net at U2.5 (TDI): now also R2.2
- new net: D3.3 (input/output_2), J13.2, R5.1, R6.2
- new net: D3.2 (input/output_1), J13.3, R7.1
- new net: C1.1, J13.6, J13.7, J13.8, J13.9
- new net: D1.2 (A), R3.2
- new net: D2.2 (A), R4.2
- no-connect marks 0 -> 3
Other:
- note added: "1 VBUS\n2 D-\n3 D+\n4 ID\n5 GND"
- note added: "6~9 Shell\n10, 11 Post"
- note added: "Config PG"
- note added: "PG"
- moved on the sheet: U2, U3, U4
