File: TE0890/local_board/mifune_TE0890_local_board.sch (KiCad schematic (older format))
At the start: 41 parts

Commit message: First prototype
Parts:
- removed D? (x8): LED, symbol Device:LED
- removed R? (x20): R, symbol Device:R
- removed SW? (x4): SW_Push, symbol Switch:SW_Push
- removed SW? (x8): SW_SPST, symbol Switch:SW_SPST
- added H1, H2, H3, H4: MountingHole, MountingHole:MountingHole_3.2mm_M3, symbol Mechanical:MountingHole
- added J1, J14, J15, J2, J3, J4, J5, J6, J7, J8: Conn_01x01, TestPoint:TestPoint_THTPad_D1.5mm_Drill0.7mm, symbol Connector_Generic:Conn_01x01
- U1: renamed from U?; footprint (none) -> TE0890:TE0890_80pin
Connections:
- net SLED3G: now reaches U1.1 (PORT_A0)
- net GND: now reaches U1.10 (GND)
- net GND: now also U1.20 (GND), U1.29 (GND), U1.30 (GND), U1.40 (GND), U1.41 (GND), U1.51 (GND), U1.52 (GND), U1.61 (GND), U1.71 (GND), U1.72 (GND), U1.9 (GND), J15.1 (Pin_1)
- net SLED2G: now reaches U1.11 (ePORT_B0)
- net SLED2F: now reaches U1.12 (PORT_B4)
- net SLED2A: now reaches U1.13 (PORT_B1)
- net SLED2B: now reaches U1.14 (PORT_B5)
- net SLED2P: now reaches U1.15 (PORT_B2)
- net SLED2C: now reaches U1.16 (PORT_B6)
- net SLED2D: now reaches U1.17 (PORT_B3)
- net SLED2E: now reaches U1.18 (PORT_B7)
- net +3V3: now reaches U1.19 (3V3)
- net +3V3: now also U1.62 (3V3)
- net SLED3F: now reaches U1.2 (PORT_A4)
- net SLED1G: now reaches U1.21 (PORT_C0)
- net SLED1F: now reaches U1.22 (PORT_C4)
- net SLED1A: now reaches U1.23 (PORT_C1)
- net SLED1B: now reaches U1.24 (PORT_C5)
- net SLED1P: now reaches U1.25 (PORT_C2)
- net SLED1C: now reaches U1.26 (PORT_C6)
- net SLED1D: now reaches U1.27 (PORT_C3)
- net SLED1E: now reaches U1.28 (PORT_C7)
- net SLED3A: now reaches U1.3 (PORT_A1)
- net SLED0G: now reaches U1.31 (PORT_D0)
- net SLED0F: now reaches U1.32 (PORT_D4)
- net SLED0A: now reaches U1.33 (PORT_D1)
- net SLED0B: now reaches U1.34 (PORT_D5)
- net SLED0P: now reaches U1.35 (PORT_D2)
- net SLED0C: now reaches U1.36 (PORT_D6)
- net SLED0D: now reaches U1.37 (PORT_D3)
- net SLED0E: now reaches U1.38 (PORT_D7)
- net +5V: now reaches U1.39 (5V)
- net +5V: now also U1.42 (5V), J14.1 (Pin_1)
- net SLED3B: now reaches U1.4 (PORT_A5)
- net TSW7: now reaches U1.43 (PORT_E7)
- net TSW6: now reaches U1.44 (PORT_E3)
- net TSW5: now reaches U1.45 (PORT_E6)
- net TSW4: now reaches U1.46 (PORT_E2)
- net LED7: now reaches U1.47 (PORT_E5)
- net LED6: now reaches U1.48 (PORT_E1)
- net LED5: now reaches U1.49 (PORT_E4)
- net SLED3P: now reaches U1.5 (PORT_A2)
- net LED4: now reaches U1.50 (PORT_E0)
- net TSW3: now reaches U1.53 (PORT_F7)
- net TSW2: now reaches U1.54 (PORT_F3)
- net TSW1: now reaches U1.55 (PORT_F6)
- net TSW0: now reaches U1.56 (PORT_F2)
- net LED3: now reaches U1.57 (PORT_F5)
- net LED2: now reaches U1.58 (PORT_F1)
- net LED1: now reaches U1.59 (PORT_F4)
- net SLED3C: now reaches U1.6 (PORT_A6)
- net LED0: now reaches U1.60 (PORT_F0)
- net at U1.63 (PORT_G7): now also J8.1 (Pin_1)
- net at U1.64 (PORT_G3): now also J7.1 (Pin_1)
- net at U1.65 (PORT_G6): now also J6.1 (Pin_1)
- net at U1.66 (PORT_G2): now also J5.1 (Pin_1)
- net at U1.67 (PORT_G5): now also J4.1 (Pin_1)
- net at U1.68 (PORT_G1): now also J3.1 (Pin_1)
- net at U1.69 (PORT_G4): now also J2.1 (Pin_1)
- net SLED3D: now reaches U1.7 (PORT_A3)
- net at U1.70 (PORT_G0): now also J1.1 (Pin_1)
- net LED11: now reaches U1.73 (PORT_H7)
- net LED10: now reaches U1.74 (PORT_H3)
- net LED9: now reaches U1.75 (PORT_H6)
- net LED8: now reaches U1.76 (PORT_H2)
- net PSW3: now reaches U1.77 (PORT_H5)
- net PSW2: now reaches U1.78 (PORT_H1)
- net PSW1: now reaches U1.79 (PORT_H4)
- net SLED3E: now reaches U1.8 (PORT_A7)
- net PSW0: now reaches U1.80 (PORT_H0)
Other:
- moved on the sheet: U1
