File: TE0890/remote_board/mifune_TE0890_remote_board.kicad_pcb (KiCad board)
At the start: 2 copper layers, 123 x 120 mm, 81 parts, among them IC1 SN74LV4T125PWR, IC2 SN74LV4T125PWR, J1 Raspberry_Pi_2_3, J10 Conn_01x01, J11 Conn_01x01, J12 Conn_01x01, J13 Conn_01x01, J14 Conn_01x01, J15 Conn_01x01, J16 Conn_01x01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

Commit message: remote board 2021 March 07
Parts:
- added J22: Conn_01x01, TestPoint:TestPoint_THTPad_D1.5mm_Drill0.7mm, F.Cu at (59.2, 105.7)
- added J23: Conn_01x01, TestPoint:TestPoint_THTPad_D1.5mm_Drill0.7mm, F.Cu at (65.3, 175.8)
- added J24: Conn_01x01, TestPoint:TestPoint_THTPad_D1.5mm_Drill0.7mm, F.Cu at (157.0, 77.5)
- added J25: Conn_01x01, TestPoint:TestPoint_THTPad_D1.5mm_Drill0.7mm, F.Cu at (155.2, 174.2)
- moved J6 12.7 mm to (150.1, 174.2)
- moved J12 7.62 mm to (150.1, 184.4)
- moved J10 7.62 mm to (150.1, 176.8)
- moved J16 7.62 mm to (143.8, 179.3)
- moved J7 7.62 mm to (150.1, 186.9)
- moved J8 5.08 mm to (150.1, 179.3)
- moved J13 5.08 mm to (143.8, 186.9)
- moved J14 5.08 mm to (143.8, 184.4)
- moved D6 4.00 mm to (47.9, 182.7)
- moved R29 4.00 mm to (53.0, 182.7)
- moved D5 3.81 mm to (47.9, 186.7)
- moved R28 3.81 mm to (53.0, 186.7)
- moved J15 2.54 mm to (143.8, 181.9)
- moved C5 1.51 mm to (58.6, 144.3), turned to 180 degrees
- moved R9 0.91 mm to (107.0, 177.2)
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Connections:
- U3 pad 39: +5VD -> +5V
- U3 pad 42: +5VD -> +5V
- U4 pad 3: +5VD -> +5V
- U6 pad 39: +5VD -> +5V
- U6 pad 42: +5VD -> +5V
Routing:
- net +5V: track 73.5 -> 324.4 mm
- net PORT_H0: track 0.00 -> 188.4 mm
- net PORT_H4: track 0.00 -> 181.5 mm
- net PORT_A0: track 0.00 -> 177.3 mm
- net PORT_H1: track 0.00 -> 174.8 mm
- net PORT_A4: track 0.00 -> 173.1 mm
- net PORT_H5: track 0.00 -> 168.7 mm
- net PORT_A1: track 0.94 -> 168.9 mm
- net PORT_A5: track 0.00 -> 164.6 mm
- net PORT_H2: track 0.00 -> 162.6 mm
- net PORT_A2: track 0.00 -> 160.4 mm
- net PORT_A6: track 0.00 -> 156.2 mm
- net PORT_H3: track 0.00 -> 155.6 mm
- net PORT_A3: track 0.00 -> 152.0 mm
- net PORT_H7: track 0.00 -> 151.3 mm
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- added copper zone on In1.Cu, net +3V3
- added copper zone on In1.Cu, net +5V
- added copper zone on In2.Cu, net GND
Other:
- copper layers 2 -> 4
- net class Default: via_dia 0.889 -> 0.5; via_drill 0.635 -> 0.2
- net class Power: via_dia 0.889 -> 0.6; via_drill 0.635 -> 0.2
- board text added: "GND"
- board text added: "mifune / rev. 0 / TE0890 / Remote Board Masayuki Takagiwa"
