File: TE0890/remote_board/mifune_TE0890_remote_board.sch (KiCad schematic (older format))
At the start: 29 parts

Commit message: 両面基板の作業途中。
Parts:
- added D5, D6: LED, LED_SMD:LED_0805_2012Metric_Pad1.15x1.40mm_HandSolder, symbol Device:LED
- added H4, H5, H6: MountingHole, MountingHole:MountingHole_2.7mm_M2.5, symbol Mechanical:MountingHole
- added J10, J11, J12, J13, J14, J15, J16, J17, J18, J19, J2, J20, J3, J4, J5, J6, J7, J8, J9: Conn_01x01, TestPoint:TestPoint_THTPad_D1.5mm_Drill0.7mm, symbol Connector_Generic:Conn_01x01
- added R20, R21, R22, R23, R29: 820, Resistor_SMD:R_0805_2012Metric_Pad1.20x1.40mm_HandSolder, symbol Device:R
- added R24, R25, R26, R27, R28: 3.9k, Resistor_SMD:R_0805_2012Metric_Pad1.20x1.40mm_HandSolder, symbol Device:R
- C1, C2, C3, C4, C5, C6: renamed from C?; footprint (none) -> Capacitor_SMD:C_0805_2012Metric_Pad1.18x1.45mm_HandSolder
- D1, D2, D3, D4: renamed from D?; footprint (none) -> LED_SMD:LED_0805_2012Metric_Pad1.15x1.40mm_HandSolder
- H1, H2, H3: renamed from H?; footprint (none) -> MountingHole:MountingHole_2.7mm_M2.5
- IC1, IC2: renamed from IC?; footprint SOP65P640X120-14N -> LibraryLoader:SOP65P640X120-14N
- J1: renamed from J?; footprint (none) -> Connector_PinHeader_2.54mm:PinHeader_2x20_P2.54mm_Vertical
- R1, R10, R11, R12, R13, R2, R3, R4, R5, R6, R7, R8, R9: renamed from R?; footprint (none) -> Resistor_SMD:R_0805_2012Metric_Pad1.20x1.40mm_HandSolder
Connections:
- net +3V3: now also R24.1, R25.1, R26.2, R27.1, R29.1
- net +5V: now also R28.1
- net GND: now also D1.1 (K), D2.1 (K), D3.1 (K), D4.1 (K), IC1.1 (1~OE), IC2.10 (3~OE), IC2.4 (2~OE), D5.1 (K), D6.1 (K); no longer IC1.10 (3~OE)
- net PI_JTAG_OE: now also IC1.10 (3~OE); no longer IC1.1 (1~OE)
- net PI_JTAG_TDI: now also R4.1; no longer R4.2
- net PI_JTAG_TDI_SRC: now also R3.1; no longer R3.2
- net PI_JTAG_TDO: now also R5.1; no longer R5.2
- net PI_JTAG_TDO_DST: now also R6.1; no longer R6.2
- net PI_RXD: now also R8.2; no longer R8.1
- net PI_RXD_DST: now also R9.2; no longer R9.1
- net PI_TXD: now also R13.2; no longer R13.1
- net PI_TXD_SRC: now also R12.2; no longer R12.1
- net GPIO17: now reaches J1.11 (GPIO17)
- net GPIO17: now also J7.1 (Pin_1)
- net SPI_CE0: now reaches J1.12 (GPIO18/PWM0)
- net SPI_CE0: now also J13.1 (Pin_1)
- net GPIO27: now reaches J1.13 (GPIO27)
- net GPIO27: now also J12.1 (Pin_1)
- net GPIO22: now reaches J1.15 (GPIO22)
- net GPIO22: now also J8.1 (Pin_1)
- net GPIO23: now reaches J1.16 (GPIO23)
- net GPIO23: now also J9.1 (Pin_1)
- net GPIO24: now reaches J1.18 (GPIO24)
- net GPIO24: now also J10.1 (Pin_1)
- net GPIO8: now reaches J1.24 (~CE0~/GPIO8)
- net GPIO8: now also J6.1 (Pin_1)
- net GPIO7: now reaches J1.26 (~CE1~/GPIO7)
- net GPIO7: now also R23.1
- net at J1.27 (ID_SD/GPIO0): now also R24.2
- net at J1.28 (ID_SC/GPIO1): now also R25.2
- net GPIO5: now reaches J1.29 (GCLK1/GPIO5)
- net GPIO5: now also R21.1
- net SDA: now reaches J1.3 (SDA/GPIO2)
- net SDA: now also J2.1 (Pin_1)
- net GPIO6: now reaches J1.31 (GCLK2/GPIO6)
- net GPIO6: now also R22.1
- net PWM0: now reaches J1.32 (PWM0/GPIO12)
- net PWM0: now also J4.1 (Pin_1)
- net PWM1: now reaches J1.33 (PWM1/GPIO13)
- net PWM1: now also J5.1 (Pin_1)
- net SPI_MISO: now reaches J1.35 (GPIO19/MISO1)
- net SPI_MISO: now also J14.1 (Pin_1)
- net GPIO26: now reaches J1.37 (GPIO26)
- net GPIO26: now also J11.1 (Pin_1)
- net SPI_MOSI: now reaches J1.38 (GPIO20/MOSI1)
- net SPI_MOSI: now also J15.1 (Pin_1)
- net SPI_SCLK: now reaches J1.40 (GPIO21/SCLK1)
- net SPI_SCLK: now also J16.1 (Pin_1)
- net SCL: now reaches J1.5 (SCL/GPIO3)
- net SCL: now also J3.1 (Pin_1)
- net GPIO4: now reaches J1.7 (GCLK0/GPIO4)
- net GPIO4: now also R20.1
- net at IC1.2 (1A): now also R12.1; no longer R1.1
- net at C1.1, R2.1: now also IC1.6 (2Y); no longer IC1.3 (1Y)
- net at IC1.5 (2A): now also R1.1; no longer R3.1
- net at IC1.8 (3Y): now also C3.1, R4.2; no longer R13.2
- net at IC1.9 (3A): now also R3.2; no longer R12.2
- net at IC2.11 (4Y): now also R6.2; no longer R9.2
- net at IC2.12 (4A): now also C2.1, R5.2; no longer R8.2
- net at IC2.3 (1Y): now also R9.1; no longer R6.1
- net at IC2.5 (2A): now also J17.1 (Pin_1), R26.1
- net at IC2.6 (2Y): now also J18.1 (Pin_1)
- net at IC2.8 (3Y): now also J20.1 (Pin_1)
- net at IC2.9 (3A): now also J19.1 (Pin_1), R27.2
- net at D1.2 (A): now also R20.2
- net at D2.2 (A): now also R21.2
- net at D3.2 (A): now also R22.2
- net at D4.2 (A): now also R23.2
- new net: IC1.3 (1Y), R13.1
- new net: IC2.2 (1A), R8.1
- new net: D6.2 (A), R29.2
- new net: D5.2 (A), R28.2
Other:
- moved on the sheet: C2, C3, C4, D1, D2, D3, D4, R1, R10, R11, R12, R13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

Commit message: remote board 2021 March 07
Parts:
- added J22, J23, J24, J25: Conn_01x01, TestPoint:TestPoint_THTPad_D1.5mm_Drill0.7mm, symbol Connector_Generic:Conn_01x01
Connections:
- net GND: now also J22.1 (Pin_1), J23.1 (Pin_1), J24.1 (Pin_1), J25.1 (Pin_1)
Changed lines of the file:
@@
 	1    0    0    -1
 $EndComp
+$Comp
+L Connector_Generic:Conn_01x01 J25
+U 1 1 60467AFC
+P 6350 6150
+F 0 "J25" H 6430 6192 50  0000 L CNN
+F 1 "Conn_01x01" H 6430 6101 50  0000 L CNN
+F 2 "TestPoint:TestPoint_THTPad_D1.5mm_Drill0.7mm" H 6350 6150 50  0001 C CNN
+F 3 "~" H 6350 6150 50  0001 C CNN
+	1    6350 6150
+	1    0    0    -1
+$EndComp
+$Comp
+L Connector_Generic:Conn_01x01 J24
+U 1 1 60467D17
+P 6350 5900
+F 0 "J24" H 6430 5942 50  0000 L CNN
+F 1 "Conn_01x01" H 6430 5851 50  0000 L CNN
+F 2 "TestPoint:TestPoint_THTPad_D1.5mm_Drill0.7mm" H 6350 5900 50  0001 C CNN
+F 3 "~" H 6350 5900 50  0001 C CNN
+	1    6350 5900
+	1    0    0    -1
+$EndComp
+$Comp
+L Connector_Generic:Conn_01x01 J23
+U 1 1 60467E87
+P 6350 5650
+F 0 "J23" H 6430 5692 50  0000 L CNN
+F 1 "Conn_01x01" H 6430 5601 50  0000 L CNN
+F 2 "TestPoint:TestPoint_THTPad_D1.5mm_Drill0.7mm" H 6350 5650 50  0001 C CNN
+F 3 "~" H 6350 5650 50  0001 C CNN
+	1    6350 5650
+	1    0    0    -1
+$EndComp
+$Comp
+L Connector_Generic:Conn_01x01 J22
+U 1 1 60467FF2
+P 6350 5400
+F 0 "J22" H 6430 5442 50  0000 L CNN
+F 1 "Conn_01x01" H 6430 5351 50  0000 L CNN
+F 2 "TestPoint:TestPoint_THTPad_D1.5mm_Drill0.7mm" H 6350 5400 50  0001 C CNN
+F 3 "~" H 6350 5400 50  0001 C CNN
+	1    6350 5400
+	1    0    0    -1
+$EndComp
+$Comp
+L power:GND #PWR022
+U 1 1 604681BD
+P 6050 6250
+F 0 "#PWR022" H 6050 6000 50  0001 C CNN
+F 1 "GND" H 6055 6077 50  0000 C CNN
+F 2 "" H 6050 6250 50  0001 C CNN
+F 3 "" H 6050 6250 50  0001 C CNN
+	1    6050 6250
+	1    0    0    -1
+$EndComp
+Wire Wire Line
+	6050 6250 6050 6150
+Wire Wire Line
+	6050 5400 6150 5400
+Wire Wire Line
+	6150 5650 6050 5650
+Connection ~ 6050 5650
+Wire Wire Line
+	6050 5650 6050 5400
+Wire Wire Line
+	6150 5900 6050 5900
+Connection ~ 6050 5900
+Wire Wire Line
+	6050 5900 6050 5650
+Wire Wire Line
+	6150 6150 6050 6150
+Connection ~ 6050 6150
+Wire Wire Line
+	6050 6150 6050 5900
 $EndSCHEMATC
