File: TE0890/remote_board/monitor.sch (KiCad schematic (older format))
At the start: 10 parts

Commit message: 両面基板の作業途中。
Parts:
- removed U?: TE0890_80P, symbol TE0890:TE0890_80P
- removed U?: TE0890_JTAG, symbol TE0890:TE0890_JTAG
- removed U?: TE0890_FTDI, symbol TE0890:TE0890_FTDI
- removed U?: TE0790_Std, symbol TE0890:TE0790_Std
- added D7: LED, LED_SMD:LED_0805_2012Metric_Pad1.15x1.40mm_HandSolder, symbol Device:LED
- added R30: 820, Resistor_SMD:R_0805_2012Metric_Pad1.20x1.40mm_HandSolder, symbol Device:R
- added U1: TE0890_JTAG, Connector_PinHeader_2.54mm:PinHeader_1x06_P2.54mm_Vertical, symbol TE0890:TE0890_JTAG
- added U2: TE0790_Std, TE0890:TE0790, symbol TE0890:TE0790_Std
- added U3: TE0890_80P, TE0890:TE0890_80pin, symbol TE0890:TE0890_80P
- added U4: TE0890_FTDI, Connector_PinHeader_2.54mm:PinHeader_1x06_P2.54mm_Vertical, symbol TE0890:TE0890_FTDI
- R14, R15, R16, R17, R18, R19: renamed from R?; footprint (none) -> Resistor_SMD:R_0805_2012Metric_Pad1.20x1.40mm_HandSolder
Connections:
- net +3.3VP: now also R30.1, U3.19 (3V3), U3.62 (3V3)
- net +5VD: now also U3.39 (5V), U3.42 (5V), U4.3 (5V0)
- net GND: now also D7.1 (K), U1.2 (GND), U2.1 (GND), U2.2 (GND), U2.GND, U3.10 (GND), U3.20 (GND), U3.29 (GND), U3.30 (GND), U3.40 (GND), U3.41 (GND), U3.51 (GND), U3.52 (GND), U3.61 (GND), U3.71 (GND), U3.72 (GND), U3.9 (GND), U4.1 (GND)
- net PI_RXD: now also U4.6 (FTDI_3)
- net PI_TXD: now also U4.5 (FTDI_2)
- net PORT_A0: now also U3.1 (PORT_A0)
- net PORT_A1: now also U3.3 (PORT_A1)
- net PORT_A2: now also U3.5 (PORT_A2)
- net PORT_A3: now also U3.7 (PORT_A3)
- net PORT_A4: now also U3.2 (PORT_A4)
- net PORT_A5: now also U3.4 (PORT_A5)
- net PORT_A6: now also U3.6 (PORT_A6)
- net PORT_A7: now also U3.8 (PORT_A7)
- net PORT_B0: now also U3.11 (ePORT_B0)
- net PORT_B1: now also U3.13 (PORT_B1)
- net PORT_B2: now also U3.15 (PORT_B2)
- net PORT_B3: now also U3.17 (PORT_B3)
- net PORT_B4: now also U3.12 (PORT_B4)
- net PORT_B5: now also U3.14 (PORT_B5)
- net PORT_B6: now also U3.16 (PORT_B6)
- net PORT_B7: now also U3.18 (PORT_B7)
- net PORT_C0: now also U3.21 (PORT_C0)
- net PORT_C1: now also U3.23 (PORT_C1)
- net PORT_C2: now also U3.25 (PORT_C2)
- net PORT_C3: now also U3.27 (PORT_C3)
- net PORT_C4: now also U3.22 (PORT_C4)
- net PORT_C5: now also U3.24 (PORT_C5)
- net PORT_C6: now also U3.26 (PORT_C6)
- net PORT_C7: now also U3.28 (PORT_C7)
- net PORT_D0: now also U3.31 (PORT_D0)
- net PORT_D1: now also U3.33 (PORT_D1)
- net PORT_D2: now also U3.35 (PORT_D2)
- net PORT_D3: now also U3.37 (PORT_D3)
- net PORT_D4: now also U3.32 (PORT_D4)
- net PORT_D5: now also U3.34 (PORT_D5)
- net PORT_D6: now also U3.36 (PORT_D6)
- net PORT_D7: now also U3.38 (PORT_D7)
- net PORT_E0: now also U3.50 (PORT_E0)
- net PORT_E1: now also U3.48 (PORT_E1)
- net PORT_E2: now also U3.46 (PORT_E2)
- net PORT_E3: now also U3.44 (PORT_E3)
- net PORT_E4: now also U3.49 (PORT_E4)
- net PORT_E5: now also U3.47 (PORT_E5)
- net PORT_E6: now also U3.45 (PORT_E6)
- net PORT_E7: now also U3.43 (PORT_E7)
- net PORT_F0: now also U3.60 (PORT_F0)
- net PORT_F1: now also U3.58 (PORT_F1)
- net PORT_F2: now also U3.56 (PORT_F2)
- net PORT_F3: now also U3.54 (PORT_F3)
- net PORT_F4: now also U3.59 (PORT_F4)
- net PORT_F5: now also U3.57 (PORT_F5)
- net PORT_F6: now also U3.55 (PORT_F6)
- net PORT_F7: now also U3.53 (PORT_F7)
- net PORT_G0: now also U3.70 (PORT_G0)
- net PORT_G1: now also U3.68 (PORT_G1)
- net PORT_G2: now also U3.66 (PORT_G2)
- net PORT_G3: now also U3.64 (PORT_G3)
- net PORT_G4: now also U3.69 (PORT_G4)
- net PORT_G5: now also U3.67 (PORT_G5)
- net PORT_G6: now also U3.65 (PORT_G6)
- net PORT_G7: now also U3.63 (PORT_G7)
- net PORT_H0: now also U3.80 (PORT_H0)
- net PORT_H1: now also U3.78 (PORT_H1)
- net PORT_H2: now also U3.76 (PORT_H2)
- net PORT_H3: now also U3.74 (PORT_H3)
- net PORT_H4: now also U3.79 (PORT_H4)
- net PORT_H5: now also U3.77 (PORT_H5)
- net PORT_H6: now also U3.75 (PORT_H6)
- net PORT_H7: now also U3.73 (PORT_H7)
- net at R14.2: now also U1.3 (TCK)
- net at R15.2: now also U1.4 (TDO)
- net at R16.2: now also U1.5 (TDI)
- net at R17.2: now also U1.6 (TMS)
- net at R18.1: now also U4.2 (FTDI_0)
- net at R19.1: now also U4.4 (FTDI_1)
- net at R16.1: now also U2.10 (TDI)
- net at R17.1: now also U2.12 (TMS)
- net at R19.2: now also U2.3 (RXD)
- net at R14.1: now also U2.4 (TCK)
- net at R18.2: now also U2.7 (TXD)
- net at R15.1: now also U2.8 (TDO)
- new net: U1.1 (3V3), U2.5 (3V3), U2.6 (VIO)
- new net: D7.2 (A), R30.2
Other:
- moved on the sheet: R14, R15, R16, R17, R18, R19

Commit message: remote board 2021 March 07
Connections:
- net +5VD renamed +5V
Changed lines of the file:
@@
 Wire Wire Line
 	4950 2900 4750 2900
-$Comp
-L power:+5VD #PWR029
-U 1 1 5F81B888
-P 6550 1000
-F 0 "#PWR029" H 6550 850 50  0001 C CNN
-F 1 "+5VD" H 6565 1173 50  0000 C CNN
-F 2 "" H 6550 1000 50  0001 C CNN
-F 3 "" H 6550 1000 50  0001 C CNN
-	1    6550 1000
-	1    0    0    -1
-$EndComp
-$Comp
-L power:+5VD #PWR022
-U 1 1 5F81C6D8
-P 4650 1000
-F 0 "#PWR022" H 4650 850 50  0001 C CNN
-F 1 "+5VD" H 4665 1173 50  0000 C CNN
-F 2 "" H 4650 1000 50  0001 C CNN
-F 3 "" H 4650 1000 50  0001 C CNN
-	1    4650 1000
-	1    0    0    -1
-$EndComp
 Wire Wire Line
 	6450 800  6450 2900
@@
 Wire Wire Line
 	4650 4900 4650 1000
-$Comp
-L power:+5VD #PWR025
-U 1 1 5F821FA1
-P 5300 6200
-F 0 "#PWR025" H 5300 6050 50  0001 C CNN
-F 1 "+5VD" H 5315 6373 50  0000 C CNN
-F 2 "" H 5300 6200 50  0001 C CNN
-F 3 "" H 5300 6200 50  0001 C CNN
-	1    5300 6200
-	1    0    0    -1
-$EndComp
 Wire Wire Line
 	5500 6500 5300 6500
@@
 Wire Wire Line
 	2750 5200 2750 5100
+$Comp
+L power:+5V #PWR0101
+U 1 1 60293DF7
+P 4650 1000
+F 0 "#PWR0101" H 4650 850 50  0001 C CNN
+F 1 "+5V" H 4665 1173 50  0000 C CNN
+F 2 "" H 4650 1000 50  0001 C CNN
+F 3 "" H 4650 1000 50  0001 C CNN
+	1    4650 1000
+	1    0    0    -1
+$EndComp
+$Comp
+L power:+5V #PWR0102
+U 1 1 60294177
+P 6550 1000
+F 0 "#PWR0102" H 6550 850 50  0001 C CNN
+F 1 "+5V" H 6565 1173 50  0000 C CNN
+F 2 "" H 6550 1000 50  0001 C CNN
+F 3 "" H 6550 1000 50  0001 C CNN
+	1    6550 1000
+	1    0    0    -1
+$EndComp
+$Comp
+L power:+5V #PWR0103
+U 1 1 6029445F
+P 5300 6200
+F 0 "#PWR0103" H 5300 6050 50  0001 C CNN
+F 1 "+5V" H 5315 6373 50  0000 C CNN
+F 2 "" H 5300 6200 50  0001 C CNN
+F 3 "" H 5300 6200 50  0001 C CNN
+	1    5300 6200
+	1    0    0    -1
+$EndComp
 $EndSCHEMATC
