File: TE0890/remote_board/user.sch (KiCad schematic (older format))
At the start: 2 parts

Commit message: 両面基板の作業途中。
Parts:
- removed U?: TE0890_80P, symbol TE0890:TE0890_80P
- removed U?: TE0890_JTAG, symbol TE0890:TE0890_JTAG
- added D8: LED, LED_SMD:LED_0805_2012Metric_Pad1.15x1.40mm_HandSolder, symbol Device:LED
- added J21: Conn_01x06, TestPoint:TestPoint_THTPad_D1.5mm_Drill0.7mm, symbol Connector_Generic:Conn_01x06
- added R31: 820, Resistor_SMD:R_0805_2012Metric_Pad1.20x1.40mm_HandSolder, symbol Device:R
- added U5: TE0890_JTAG, Connector_PinHeader_2.54mm:PinHeader_1x06_P2.54mm_Vertical, symbol TE0890:TE0890_JTAG
- added U6: TE0890_80P, TE0890:TE0890_80pin, symbol TE0890:TE0890_80P
- added U7: TE0890_FTDI, Connector_PinHeader_2.54mm:PinHeader_1x06_P2.54mm_Vertical, symbol TE0890:TE0890_FTDI
Connections:
- net +3.3VA: now also R31.1, U5.1 (3V3), U6.19 (3V3), U6.62 (3V3)
- net +5VD: now also U6.39 (5V), U6.42 (5V)
- net GND: now also D8.1 (K), U5.2 (GND), U6.10 (GND), U6.20 (GND), U6.29 (GND), U6.30 (GND), U6.40 (GND), U6.41 (GND), U6.51 (GND), U6.52 (GND), U6.61 (GND), U6.71 (GND), U6.72 (GND), U6.9 (GND)
- net PI_JTAG_TCK: now also U5.3 (TCK)
- net PI_JTAG_TDI: now also U5.5 (TDI)
- net PI_JTAG_TDO: now also U5.4 (TDO)
- net PI_JTAG_TMS: now also U5.6 (TMS)
- net PORT_A0: now also U6.1 (PORT_A0)
- net PORT_A1: now also U6.3 (PORT_A1)
- net PORT_A2: now also U6.5 (PORT_A2)
- net PORT_A3: now also U6.7 (PORT_A3)
- net PORT_A4: now also U6.2 (PORT_A4)
- net PORT_A5: now also U6.4 (PORT_A5)
- net PORT_A6: now also U6.6 (PORT_A6)
- net PORT_A7: now also U6.8 (PORT_A7)
- net PORT_B0: now also U6.11 (ePORT_B0)
- net PORT_B1: now also U6.13 (PORT_B1)
- net PORT_B2: now also U6.15 (PORT_B2)
- net PORT_B3: now also U6.17 (PORT_B3)
- net PORT_B4: now also U6.12 (PORT_B4)
- net PORT_B5: now also U6.14 (PORT_B5)
- net PORT_B6: now also U6.16 (PORT_B6)
- net PORT_B7: now also U6.18 (PORT_B7)
- net PORT_C0: now also U6.21 (PORT_C0)
- net PORT_C1: now also U6.23 (PORT_C1)
- net PORT_C2: now also U6.25 (PORT_C2)
- net PORT_C3: now also U6.27 (PORT_C3)
- net PORT_C4: now also U6.22 (PORT_C4)
- net PORT_C5: now also U6.24 (PORT_C5)
- net PORT_C6: now also U6.26 (PORT_C6)
- net PORT_C7: now also U6.28 (PORT_C7)
- net PORT_D0: now also U6.31 (PORT_D0)
- net PORT_D1: now also U6.33 (PORT_D1)
- net PORT_D2: now also U6.35 (PORT_D2)
- net PORT_D3: now also U6.37 (PORT_D3)
- net PORT_D4: now also U6.32 (PORT_D4)
- net PORT_D5: now also U6.34 (PORT_D5)
- net PORT_D6: now also U6.36 (PORT_D6)
- net PORT_D7: now also U6.38 (PORT_D7)
- net PORT_E0: now also U6.50 (PORT_E0)
- net PORT_E1: now also U6.48 (PORT_E1)
- net PORT_E2: now also U6.46 (PORT_E2)
- net PORT_E3: now also U6.44 (PORT_E3)
- net PORT_E4: now also U6.49 (PORT_E4)
- net PORT_E5: now also U6.47 (PORT_E5)
- net PORT_E6: now also U6.45 (PORT_E6)
- net PORT_E7: now also U6.43 (PORT_E7)
- net PORT_F0: now also U6.60 (PORT_F0)
- net PORT_F1: now also U6.58 (PORT_F1)
- net PORT_F2: now also U6.56 (PORT_F2)
- net PORT_F3: now also U6.54 (PORT_F3)
- net PORT_F4: now also U6.59 (PORT_F4)
- net PORT_F5: now also U6.57 (PORT_F5)
- net PORT_F6: now also U6.55 (PORT_F6)
- net PORT_F7: now also U6.53 (PORT_F7)
- net PORT_G0: now also U6.70 (PORT_G0)
- net PORT_G1: now also U6.68 (PORT_G1)
- net PORT_G2: now also U6.66 (PORT_G2)
- net PORT_G3: now also U6.64 (PORT_G3)
- net PORT_G4: now also U6.69 (PORT_G4)
- net PORT_G5: now also U6.67 (PORT_G5)
- net PORT_G6: now also U6.65 (PORT_G6)
- net PORT_G7: now also U6.63 (PORT_G7)
- net PORT_H0: now also U6.80 (PORT_H0)
- net PORT_H1: now also U6.78 (PORT_H1)
- net PORT_H2: now also U6.76 (PORT_H2)
- net PORT_H3: now also U6.74 (PORT_H3)
- net PORT_H4: now also U6.79 (PORT_H4)
- net PORT_H5: now also U6.77 (PORT_H5)
- net PORT_H6: now also U6.75 (PORT_H6)
- net PORT_H7: now also U6.73 (PORT_H7)
- new net: J21.1 (Pin_1), U7.1 (GND)
- new net: J21.2 (Pin_2), U7.2 (FTDI_0)
- new net: J21.3 (Pin_3), U7.3 (5V0)
- new net: J21.4 (Pin_4), U7.4 (FTDI_1)
- new net: J21.5 (Pin_5), U7.5 (FTDI_2)
- new net: J21.6 (Pin_6), U7.6 (FTDI_3)
- new net: D8.2 (A), R31.2
Changed lines of the file:
@@
 $EndDescr
-$Comp
-L TE0890:TE0890_80P U?
-U 1 1 5F82A65F
-P 5550 3350
-AR Path="/5F7AA1FC/5F82A65F" Ref="U?"  Part="1"
-AR Path="/5F7AA2D2/5F82A65F" Ref="U?"  Part="1"
-F 0 "U?" H 5550 5515 50  0000 C CNN
-F 1 "TE0890_80P" H 5550 5424 50  0000 C CNN
-F 2 "" H 5550 3350 50  0001 C CNN
-F 3 "" H 5550 3350 50  0001 C CNN
-	1    5550 3350
-	1    0    0    -1
-$EndComp
 $Comp
 L power:GND #PWR?
@@
 P 4800 5450
 AR Path="/5F7AA1FC/5F82A665" Ref="#PWR?"  Part="1"
-AR Path="/5F7AA2D2/5F82A665" Ref="#PWR?"  Part="1"
-F 0 "#PWR?" H 4800 5200 50  0001 C CNN
+AR Path="/5F7AA2D2/5F82A665" Ref="#PWR034"  Part="1"
+F 0 "#PWR034" H 4800 5200 50  0001 C CNN
 F 1 "GND" H 4805 5277 50  0000 C CNN
 F 2 "" H 4800 5450 50  0001 C CNN
@@
 P 6300 5450
 AR Path="/5F7AA1FC/5F82A66B" Ref="#PWR?"  Part="1"
-AR Path="/5F7AA2D2/5F82A66B" Ref="#PWR?"  Part="1"
-F 0 "#PWR?" H 6300 5200 50  0001 C CNN
+AR Path="/5F7AA2D2/5F82A66B" Ref="#PWR035"  Part="1"
+F 0 "#PWR035" H 6300 5200 50  0001 C CNN
 F 1 "GND" H 6305 5277 50  0000 C CNN
 F 2 "" H 6300 5450 50  0001 C CNN
@@
 P 6500 1350
 AR Path="/5F7AA1FC/5F82A6A1" Ref="#PWR?"  Part="1"
-AR Path="/5F7AA2D2/5F82A6A1" Ref="#PWR?"  Part="1"
-F 0 "#PWR?" H 6500 1200 50  0001 C CNN
+AR Path="/5F7AA2D2/5F82A6A1" Ref="#PWR037"  Part="1"
+F 0 "#PWR037" H 6500 1200 50  0001 C CNN
 F 1 "+5VD" H 6515 1523 50  0000 C CNN
 F 2 "" H 6500 1350 50  0001 C CNN
@@
 P 4600 1350
 AR Path="/5F7AA1FC/5F82A6A7" Ref="#PWR?"  Part="1"
-AR Path="/5F7AA2D2/5F82A6A7" Ref="#PWR?"  Part="1"
-F 0 "#PWR?" H 4600 1200 50  0001 C CNN
+AR Path="/5F7AA2D2/5F82A6A7" Ref="#PWR032"  Part="1"
+F 0 "#PWR032" H 4600 1200 50  0001 C CNN
 F 1 "+5VD" H 4615 1523 50  0000 C CNN
 F 2 "" H 4600 1350 50  0001 C CNN
@@
 	4600 5250 4600 1350
 $Comp
-L TE0890:TE0890_JTAG U?
-U 1 1 5F82F8FB
-P 3000 6800
-AR Path="/5F7AA1FC/5F82F8FB" Ref="U?"  Part="1"
-AR Path="/5F7AA2D2/5F82F8FB" Ref="U?"  Part="1"
-F 0 "U?" H 3228 6851 50  0000 L CNN
-F 1 "TE0890_JTAG" H 3228 6760 50  0000 L CNN
-F 2 "" H 3000 6800 50  0001 C CNN
-F 3 "" H 3000 6800 50  0001 C CNN
-	1    3000 6800
-	1    0    0    -1
-$EndComp
-$Comp
 L power:GND #PWR?
 U 1 1 5F82F945
-P 2600 7150
+P 2150 7150
 AR Path="/5F7AA1FC/5F82F945" Ref="#PWR?"  Part="1"
-AR Path="/5F7AA2D2/5F82F945" Ref="#PWR?"  Part="1"
-F 0 "#PWR?" H 2600 6900 50  0001 C CNN
-F 1 "GND" H 2605 6977 50  0000 C CNN
-F 2 "" H 2600 7150 50  0001 C CNN
-F 3 "" H 2600 7150 50  0001 C CNN
-	1    2600 7150
-	1    0    0    -1
-$EndComp
-Text GLabel 2500 6750 0    50   Input ~ 0
+AR Path="/5F7AA2D2/5F82F945" Ref="#PWR031"  Part="1"
+F 0 "#PWR031" H 2150 6900 50  0001 C CNN
+F 1 "GND" H 2155 6977 50  0000 C CNN
+F 2 "" H 2150 7150 50  0001 C CNN
+F 3 "" H 2150 7150 50  0001 C CNN
+	1    2150 7150
+	1    0    0    -1
+$EndComp
+Text GLabel 2050 6750 0    50   Input ~ 0
 PI_JTAG_TCK
-Text GLabel 2500 6950 0    50   Input ~ 0
+Text GLabel 2050 6950 0    50   Input ~ 0
 PI_JTAG_TDI
-Text GLabel 2500 7050 0    50   Input ~ 0
+Text GLabel 2050 7050 0    50   Input ~ 0
 PI_JTAG_TMS
-Text GLabel 2500 6850 0    50   Output ~ 0
+Text GLabel 2050 6850 0    50   Output ~ 0
 PI_JTAG_TDO
 $Comp
-L power:+3.3VA #PWR?
+L power:+3.3VA #PWR033
 U 1 1 5F837BEF
 P 4700 1150
-F 0 "#PWR?" H 4700 1000 50  0001 C CNN
+F 0 "#PWR033" H 4700 1000 50  0001 C CNN
 F 1 "+3.3VA" H 4715 1323 50  0000 C CNN
 F 2 "" H 4700 1150 50  0001 C CNN
@@
 $EndComp
 $Comp
-L power:+3.3VA #PWR?
+L power:+3.3VA #PWR036
 U 1 1 5F837EE4
 P 6400 1150
-F 0 "#PWR?" H 6400 1000 50  0001 C CNN
+F 0 "#PWR036" H 6400 1000 50  0001 C CNN
 F 1 "+3.3VA" H 6415 1323 50  0000 C CNN
 F 2 "" H 6400 1150 50  0001 C CNN
@@
 $EndComp
 $Comp
-L power:+3.3VA #PWR?
+L power:+3.3VA #PWR030
 U 1 1 5F83845B
-P 2600 6450
-F 0 "#PWR?" H 2600 6300 50  0001 C CNN
-F 1 "+3.3VA" H 2615 6623 50  0000 C CNN
-F 2 "" H 2600 6450 50  0001 C CNN
-F 3 "" H 2600 6450 50  0001 C CNN
-	1    2600 6450
-	1    0    0    -1
-$EndComp
-Wire Wire Line
-	2700 6550 2600 6550
-Wire Wire Line
-	2600 6550 2600 6450
-Wire Wire Line
-	2700 6650 2600 6650
-Wire Wire Line
-	2600 6650 2600 7150
-Wire Wire Line
-	2700 7050 2500 7050
-Wire Wire Line
-	2500 6950 2700 6950
-Wire Wire Line
-	2700 6850 2500 6850
-Wire Wire Line
-	2500 6750 2700 6750
-Text Notes 3000 7250 0    50   ~ 0
+P 2150 6450
+F 0 "#PWR030" H 2150 6300 50  0001 C CNN
+F 1 "+3.3VA" H 2165 6623 50  0000 C CNN
+F 2 "" H 2150 6450 50  0001 C CNN
+F 3 "" H 2150 6450 50  0001 C CNN
+	1    2150 6450
+	1    0    0    -1
+$EndComp
+Wire Wire Line
+	2250 6550 2150 6550
+Wire Wire Line
+	2150 6550 2150 6450
+Wire Wire Line
+	2250 6650 2150 6650
+Wire Wire Line
+	2150 6650 2150 7150
+Wire Wire Line
+	2250 7050 2050 7050
+Wire Wire Line
+	2050 6950 2250 6950
+Wire Wire Line
+	2250 6850 2050 6850
+Wire Wire Line
+	2050 6750 2250 6750
+Text Notes 2550 7250 0    50   ~ 0
 Write default image into on-board flash via another JTAG cable.
 Text GLabel 4400 1450 0    50   UnSpc ~ 0
@@
 Wire Wire Line
 	6200 5150 6700 5150
+$Comp
+L TE0890:TE0890_80P U6
+U 1 1 5FF48834
+P 5550 3350
+F 0 "U6" H 5550 5515 50  0000 C CNN
+F 1 "TE0890_80P" H 5550 5424 50  0000 C CNN
+F 2 "TE0890:TE0890_80pin" H 5550 3350 50  0001 C CNN
+F 3 "" H 5550 3350 50  0001 C CNN
+	1    5550 3350
+	1    0    0    -1
+$EndComp
+$Comp
+L TE0890:TE0890_JTAG U5
+U 1 1 5FF4A328
+P 2550 6800
+F 0 "U5" H 2778 6851 50  0000 L CNN
+F 1 "TE0890_JTAG" H 2778 6760 50  0000 L CNN
+F 2 "Connector_PinHeader_2.54mm:PinHeader_1x06_P2.54mm_Vertical" H 2550 6800 50  0001 C CNN
+F 3 "" H 2550 6800 50  0001 C CNN
+	1    2550 6800
+	1    0    0    -1
+$EndComp
+$Comp
+L TE0890:TE0890_FTDI U7
+U 1 1 5FF4DA6C
+P 2600 5450
+F 0 "U7" H 2878 5501 50  0000 L CNN
+F 1 "TE0890_FTDI" H 2878 5410 50  0000 L CNN
+F 2 "Connector_PinHeader_2.54mm:PinHeader_1x06_P2.54mm_Vertical" H 2250 5450 50  0001 C CNN
+F 3 "" H 2250 5450 50  0001 C CNN
+	1    2600 5450
+	1    0    0    -1
+$EndComp
+$Comp
+L Connector_Generic:Conn_01x06 J21
+U 1 1 603013ED
+P 2500 4550
+F 0 "J21" H 2580 4542 50  0000 L CNN
+F 1 "Conn_01x06" H 2580 4451 50  0000 L CNN
+F 2 "TestPoint:TestPoint_THTPad_D1.5mm_Drill0.7mm" H 2500 4550 50  0001 C CNN
+F 3 "~" H 2500 4550 50  0001 C CNN
+	1    2500 4550
+	1    0    0    -1
+$EndComp
+Wire Wire Line
+	2250 5200 2150 5200
+Wire Wire Line
+	2150 5200 2150 4350
+Wire Wire Line
+	2150 4350 2300 4350
+Wire Wire Line
+	2300 4450 2050 4450
+Wire Wire Line
+	2050 4450 2050 5300
+Wire Wire Line
+	2050 5300 2250 5300
+Wire Wire Line
+	2250 5400 1950 5400
+Wire Wire Line
+	1950 5400 1950 4550
+Wire Wire Line
+	1950 4550 2300 4550
+Wire Wire Line
+	2300 4650 1850 4650
+Wire Wire Line
+	1850 4650 1850 5500
+Wire Wire Line
+	1850 5500 2250 5500
+Wire Wire Line
+	2250 5600 1750 5600
+Wire Wire Line
+	1750 5600 1750 4750
+Wire Wire Line
+	1750 4750 2300 4750
+Wire Wire Line
+	2300 4850 1650 4850
+Wire Wire Line
+	1650 5700 2250 5700
+Wire Wire Line
+	1650 4850 1650 5700
+$Comp
+L Device:LED D?
+U 1 1 60550082
+P 8600 5650
+AR Path="/60550082" Ref="D?"  Part="1"
+AR Path="/5F7AA2D2/60550082" Ref="D8"  Part="1"
+F 0 "D8" H 8400 5700 50  0000 C CNN
+F 1 "LED" H 8800 5700 50  0000 C CNN
+F 2 "LED_SMD:LED_0805_2012Metric_Pad1.15x1.40mm_HandSolder" H 8600 5650 50  0001 C CNN
+F 3 "~" H 8600 5650 50  0001 C CNN
+	1    8600 5650
+	1    0    0    -1
+$EndComp
+$Comp
+L Device:R R?
+U 1 1 60550088
+P 9300 5650
+AR Path="/60550088" Ref="R?"  Part="1"
+AR Path="/5F7AA2D2/60550088" Ref="R31"  Part="1"
+F 0 "R31" V 9250 5400 50  0000 C CNN
+F 1 "820" V 9250 5900 50  0000 C CNN
+F 2 "Resistor_SMD:R_0805_2012Metric_Pad1.20x1.40mm_HandSolder" V 9230 5650 50  0001 C CNN
+F 3 "~" H 9300 5650 50  0001 C CNN
+	1    9300 5650
+	0    1    1    0
+$EndComp
+Wire Wire Line
+	8750 5650 9150 5650
+$Comp
+L power:GND #PWR?
+U 1 1 605557FB
+P 8350 5750
+AR Path="/5F7AA1FC/605557FB" Ref="#PWR?"  Part="1"
+AR Path="/5F7AA2D2/605557FB" Ref="#PWR047"  Part="1"
+F 0 "#PWR047" H 8350 5500 50  0001 C CNN
+F 1 "GND" H 8355 5577 50  0000 C CNN
+F 2 "" H 8350 5750 50  0001 C CNN
+F 3 "" H 8350 5750 50  0001 C CNN
+	1    8350 5750
+	1    0    0    -1
+$EndComp
+$Comp
+L power:+3.3VA #PWR048
+U 1 1 605559CA
+P 9700 5600
+F 0 "#PWR048" H 9700 5450 50  0001 C CNN
+F 1 "+3.3VA" H 9715 5773 50  0000 C CNN
+F 2 "" H 9700 5600 50  0001 C CNN
+F 3 "" H 9700 5600 50  0001 C CNN
+	1    9700 5600
+	1    0    0    -1
+$EndComp
+Wire Wire Line
+	8450 5650 8350 5650
+Wire Wire Line
+	8350 5650 8350 5750
+Wire Wire Line
+	9450 5650 9700 5650
+Wire Wire Line
+	9700 5650 9700 5600
 $EndSCHEMATC

Commit message: remote board 2021 March 07
Connections:
- net +5VD renamed +5V
Changed lines of the file:
@@
 Wire Wire Line
 	4900 3250 4700 3250
-$Comp
-L power:+5VD #PWR?
-U 1 1 5F82A6A1
-P 6500 1350
-AR Path="/5F7AA1FC/5F82A6A1" Ref="#PWR?"  Part="1"
-AR Path="/5F7AA2D2/5F82A6A1" Ref="#PWR037"  Part="1"
-F 0 "#PWR037" H 6500 1200 50  0001 C CNN
-F 1 "+5VD" H 6515 1523 50  0000 C CNN
-F 2 "" H 6500 1350 50  0001 C CNN
-F 3 "" H 6500 1350 50  0001 C CNN
-	1    6500 1350
-	1    0    0    -1
-$EndComp
-$Comp
-L power:+5VD #PWR?
-U 1 1 5F82A6A7
-P 4600 1350
-AR Path="/5F7AA1FC/5F82A6A7" Ref="#PWR?"  Part="1"
-AR Path="/5F7AA2D2/5F82A6A7" Ref="#PWR032"  Part="1"
-F 0 "#PWR032" H 4600 1200 50  0001 C CNN
-F 1 "+5VD" H 4615 1523 50  0000 C CNN
-F 2 "" H 4600 1350 50  0001 C CNN
-F 3 "" H 4600 1350 50  0001 C CNN
-	1    4600 1350
-	1    0    0    -1
-$EndComp
 Wire Wire Line
 	6400 1150 6400 3250
@@
 Wire Wire Line
 	9700 5650 9700 5600
+$Comp
+L power:+5V #PWR0104
+U 1 1 602957E9
+P 6500 1350
+F 0 "#PWR0104" H 6500 1200 50  0001 C CNN
+F 1 "+5V" H 6515 1523 50  0000 C CNN
+F 2 "" H 6500 1350 50  0001 C CNN
+F 3 "" H 6500 1350 50  0001 C CNN
+	1    6500 1350
+	1    0    0    -1
+$EndComp
+$Comp
+L power:+5V #PWR0105
+U 1 1 60295BFF
+P 4600 1350
+F 0 "#PWR0105" H 4600 1200 50  0001 C CNN
+F 1 "+5V" H 4615 1523 50  0000 C CNN
+F 2 "" H 4600 1350 50  0001 C CNN
+F 3 "" H 4600 1350 50  0001 C CNN
+	1    4600 1350
+	1    0    0    -1
+$EndComp
 $EndSCHEMATC
